File: PCBs/drive_V2/iprld.kicad_sch (KiCad schematic)
At the start: 77 parts, among them IC1 W25Q16JVUXIQ_TR, IC2 ADS1115IDGSR, J1 TYPE-C-31-M-12, U1 AMS1117-3.3, U11 4N35, U12 4N35, U13 4N35, U14 4N35, U2 ESP32-S3, U3 4N35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

Commit message: added more decoupling capacitors, fixed flash connections, clock capacitors, thick power traces
Parts:
- added C13, C18, C19, C20: 0.1u, Capacitor_SMD:C_0603_1608Metric, symbol Device:C
- C16: value 12p -> 14p
- C17: value 15p -> 14p
Connections:
- net +3.3V: now also C13.2, C18.2, C19.2, C20.2
- net GND: now also C13.1, C18.1, C19.1, C20.1
- net SPID: now also IC1.5 (DI(IO0)); no longer IC1.2 (DO(IO1))
- net SPIQ: now also IC1.2 (DO(IO1)); no longer IC1.5 (DI(IO0))
