File: PCBs/Power_PCB/Power_PCB/Current_sensing.kicad_sch (KiCad schematic)
At the start: 25 parts, among them IC1 ADS1115BQDGSRQ1, IC10 ACS712ELCTR-20A-T, IC2 ADS1115BQDGSRQ1, IC7 ACS712ELCTR-20A-T, IC8 ACS712ELCTR-20A-T, IC9 ACS712ELCTR-20A-T

Commit message: Second iteration power board
Connections:
- net ARM_READ: now also IC2.4 (AIN0); no longer IC1.7 (AIN3)
- net COMMS_READ: now also IC1.6 (AIN2); no longer IC2.4 (AIN0)
- net DRILL_READ: now also IC1.7 (AIN3); no longer IC1.6 (AIN2)
Changed lines of the file:
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@@
 	(label "COMMS_V"
 		(at 201.93 128.27 0)
-		(fields_autoplaced yes)
 		(effects
 			(font
@@
 	(label "SCL"
 		(at 139.7 57.15 180)
-		(fields_autoplaced yes)
-		(effects
-			(font
-				(size 1.27 1.27)
-			)
-			(justify right bottom)
+		(effects
+			(font
+				(size 1.27 1.27)
+			)
+			(justify right bottom)
+		)
+	)
+	(label "DRILL_READ"
+		(at 138.43 64.77 0)
+		(effects
+			(font
+				(size 1.27 1.27)
+			)
+			(justify left bottom)
 		)
 	)
 	(label "SCL"
 		(at 208.28 55.88 0)
-		(fields_autoplaced yes)
 		(effects
 			(font
@@
 	(label "14V8_PROTECTED"
 		(at 68.58 92.71 180)
-		(fields_autoplaced yes)
 		(effects
 			(font
@@
 	(label "SCL"
 		(at 254 95.25 180)
-		(fields_autoplaced yes)
 		(effects
 			(font
@@
 	(label "14V8_PROTECTED"
 		(at 21.59 76.2 180)
-		(fields_autoplaced yes)
 		(effects
 			(font
@@
 	(label "ARM_READ"
 		(at 236.22 101.6 0)
-		(fields_autoplaced yes)
 		(effects
 			(font
@@
 	(label "14V8_COMMS_OUT"
 		(at 165.1 132.08 180)
-		(fields_autoplaced yes)
 		(effects
 			(font
@@
 	(label "SDA"
 		(at 208.28 58.42 0)
-		(fields_autoplaced yes)
-		(effects
-			(font
-				(size 1.27 1.27)
-			)
-			(justify left bottom)
-		)
-	)
-	(label "COMMS_READ"
-		(at 161.29 63.5 0)
-		(fields_autoplaced yes)
-		(effects
-			(font
-				(size 1.27 1.27)
-			)
-			(justify left bottom)
-		)
-	)
-	(label "ARM_READ"
-		(at 138.43 64.77 0)
-		(fields_autoplaced yes)
 		(effects
 			(font
@@
 	(label "14V8_DRILL_OUT"
 		(at 68.58 97.79 180)
-		(fields_autoplaced yes)
 		(effects
 			(font
@@
 	(label "DRILL_V"
 		(at 105.41 93.98 0)
-		(fields_autoplaced yes)
 		(effects
 			(font
@@
 	(label "14V8_PROTECTED"
 		(at 73.66 52.07 180)
-		(fields_autoplaced yes)
 		(effects
 			(font
@@
 	(label "COMMS_READ"
 		(at 234.95 135.89 0)
-		(fields_autoplaced yes)
 		(effects
 			(font
@@
 	(label "14V8_COMMS_OUT"
 		(at 254 107.95 180)
-		(fields_autoplaced yes)
+		(effects
+			(font
+				(size 1.27 1.27)
+			)
+			(justify right bottom)
+		)
+	)
+	(label "ARM_V"
+		(at 203.2 93.98 0)
+		(effects
+			(font
+				(size 1.27 1.27)
+			)
+			(justify left bottom)
+		)
+	)
+	(label "14V8_DRIVE_OUT"
+		(at 254 105.41 180)
+		(effects
+			(font
+				(size 1.27 1.27)
+			)
+			(justify right bottom)
+		)
+	)
+	(label "DRIVE_V"
+		(at 105.41 128.27 0)
+		(effects
+			(font
+				(size 1.27 1.27)
+			)
+			(justify left bottom)
+		)
+	)
+	(label "14V8_PROTECTED"
+		(at 165.1 127 180)
+		(effects
+			(font
+				(size 1.27 1.27)
+			)
+			(justify right bottom)
+		)
+	)
+	(label "SDA"
+		(at 254 97.79 180)
+		(effects
+			(font
+				(size 1.27 1.27)
+			)
+			(justify right bottom)
+		)
+	)
+	(label "14V8_ARM_OUT"
+		(at 166.37 97.79 180)
+		(effects
+			(font
+				(size 1.27 1.27)
+			)
+			(justify right bottom)
+		)
+	)
+	(label "14V8_ARM_OUT"
+		(at 254 100.33 180)
+		(effects
+			(font
+				(size 1.27 1.27)
+			)
+			(justify right bottom)
+		)
+	)
+	(label "SDA"
+		(at 139.7 59.69 180)
+		(effects
+			(font
+				(size 1.27 1.27)
+			)
+			(justify right bottom)
+		)
+	)
+	(label "ARM_READ"
+		(at 161.29 63.5 0)
+		(effects
+			(font
+				(size 1.27 1.27)
+			)
+			(justify left bottom)
+		)
+	)
+	(label "DRILL_READ"
+		(at 138.43 101.6 0)
+		(effects
+			(font
+				(size 1.27 1.27)
+			)
+			(justify left bottom)
+		)
+	)
+	(label "14V8_DRIVE_OUT"
+		(at 68.58 132.08 180)
+		(effects
+			(font
+				(size 1.27 1.27)
+			)
+			(justify right bottom)
+		)
+	)
+	(label "14V8_PROTECTED"
+		(at 68.58 127 180)
+		(effects
+			(font
+				(size 1.27 1.27)
+			)
+			(justify right bottom)
+		)
+	)
+	(label "14V8_PROTECTED"
+		(at 166.37 92.71 180)
+		(effects
+			(font
+				(size 1.27 1.27)
+			)
+			(justify right bottom)
+		)
+	)
+	(label "DRIVE_READ"
+		(at 138.43 135.89 0)
+		(effects
+			(font
+				(size 1.27 1.27)
+			)
+			(justify left bottom)
+		)
+	)
+	(label "COMMS_READ"
+		(at 134.62 67.31 0)
+		(effects
+			(font
+				(size 1.27 1.27)
+			)
+			(justify left bottom)
+		)
+	)
+	(label "14V8_DRILL_OUT"
+		(at 254 102.87 180)
 		(effects
 			(font
@@
 	(label "DRIVE_READ"
 		(at 161.29 66.04 0)
-		(fields_autoplaced yes)
-		(effects
-			(font
-				(size 1.27 1.27)
-			)
-			(justify left bottom)
-		)
-	)
-	(label "ARM_V"
-		(at 203.2 93.98 0)
-		(fields_autoplaced yes)
-		(effects
-			(font
-				(size 1.27 1.27)
-			)
-			(justify left bottom)
-		)
-	)
-	(label "14V8_DRIVE_OUT"
-		(at 254 105.41 180)
-		(fields_autoplaced yes)
-		(effects
-			(font
-				(size 1.27 1.27)
-			)
-			(justify right bottom)
-		)
-	)
-	(label "DRIVE_V"
-		(at 105.41 128.27 0)
-		(fields_autoplaced yes)
-		(effects
-			(font
-				(size 1.27 1.27)
-			)
-			(justify left bottom)
-		)
-	)
-	(label "14V8_PROTECTED"
-		(at 165.1 127 180)
-		(fields_autoplaced yes)
-		(effects
-			(font
-				(size 1.27 1.27)
-			)
-			(justify right bottom)
-		)
-	)
-	(label "SDA"
-		(at 254 97.79 180)
-		(fields_autoplaced yes)
-		(effects
-			(font
-				(size 1.27 1.27)
-			)
-			(justify right bottom)
-		)
-	)
-	(label "14V8_ARM_OUT"
-		(at 166.37 97.79 180)
-		(fields_autoplaced yes)
-		(effects
-			(font
-				(size 1.27 1.27)
-			)
-			(justify right bottom)
-		)
-	)
-	(label "14V8_ARM_OUT"
-		(at 254 100.33 180)
-		(fields_autoplaced yes)
-		(effects
-			(font
-				(size 1.27 1.27)
-			)
-			(justify right bottom)
-		)
-	)
-	(label "SDA"
-		(at 139.7 59.69 180)
-		(fields_autoplaced yes)
-		(effects
-			(font
-				(size 1.27 1.27)
-			)
-			(justify right bottom)
-		)
-	)
-	(label "DRILL_READ"
-		(at 138.43 101.6 0)
-		(fields_autoplaced yes)
-		(effects
-			(font
-				(size 1.27 1.27)
-			)
-			(justify left bottom)
-		)
-	)
-	(label "14V8_DRIVE_OUT"
-		(at 68.58 132.08 180)
-		(fields_autoplaced yes)
-		(effects
-			(font
-				(size 1.27 1.27)
-			)
-			(justify right bottom)
-		)
-	)
-	(label "DRILL_READ"
-		(at 134.62 67.31 0)
-		(fields_autoplaced yes)
-		(effects
-			(font
-				(size 1.27 1.27)
-			)
-			(justify left bottom)
-		)
-	)
-	(label "14V8_PROTECTED"
-		(at 68.58 127 180)
-		(fields_autoplaced yes)
-		(effects
-			(font
-				(size 1.27 1.27)
-			)
-			(justify right bottom)
-		)
-	)
-	(label "14V8_PROTECTED"
-		(at 166.37 92.71 180)
-		(fields_autoplaced yes)
-		(effects
-			(font
-				(size 1.27 1.27)
-			)
-			(justify right bottom)
-		)
-	)
-	(label "DRIVE_READ"
-		(at 138.43 135.89 0)
-		(fields_autoplaced yes)
-		(effects
-			(font
-				(size 1.27 1.27)
-			)
-			(justify left bottom)
-		)
-	)
-	(label "14V8_DRILL_OUT"
-		(at 254 102.87 180)
-		(fields_autoplaced yes)
-		(effects
-			(font
-				(size 1.27 1.27)
-			)
-			(justify right bottom)
+		(effects
+			(font
+				(size 1.27 1.27)
+			)
+			(justify left bottom)
 		)
 	)
@@
 		(shape output)
 		(at 261.62 102.87 0)
-		(fields_autoplaced yes)
 		(effects
 			(font
@@
 		(shape output)
 		(at 261.62 97.79 0)
-		(fields_autoplaced yes)
 		(effects
 			(font
@@
 		(shape output)
 		(at 261.62 107.95 0)
-		(fields_autoplaced yes)
 		(effects
 			(font
@@
 		(shape output)
 		(at 261.62 105.41 0)
-		(fields_autoplaced yes)
 		(effects
 			(font
@@
 		(shape output)
 		(at 261.62 95.25 0)
-		(fields_autoplaced yes)
 		(effects
 			(font
@@
 		(shape output)
 		(at 261.62 100.33 0)
-		(fields_autoplaced yes)
 		(effects
 			(font
@@
 		(shape input)
 		(at 27.94 76.2 0)
-		(fields_autoplaced yes)
-		(effects
-			(font
+		(effects
+			(font
