File: PCBs/Power_V2_main/Sensing.kicad_sch (KiCad schematic)
At the start: 8 parts, among them IC2 ADS1115BQDGSRQ1, IC3 ADS1115BQDGSRQ1, J11 Conn_01x04, J13 Conn_01x04, J14 Conn_01x04

Commit message: shortened main board and secondary
Parts:
- IC2, IC3: footprint IPRL_footprints:SOP50P490X110-10N -> iprl_footprints:SOP50P490X110-10N
Changed lines of the file:
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@@
-	(wire
-		(pts
-			(xy 38.1 180.34) (xy 45.72 180.34)
-		)
-		(stroke
-			(width 0)
-			(type default)
-		)
-	)
 	(wire
 		(pts
@@
 	(wire
 		(pts
-			(xy 38.1 172.72) (xy 45.72 172.72)
-		)
-		(stroke
-			(width 0)
-			(type default)
-		)
-	)
-	(wire
-		(pts
-			(xy 38.1 185.42) (xy 45.72 185.42)
+			(xy 82.55 187.96) (xy 90.17 187.96)
+		)
+		(stroke
+			(width 0)
+			(type default)
+		)
+	)
+	(wire
+		(pts
+			(xy 83.82 171.45) (xy 90.17 171.45)
 		)
 		(stroke
@@
 	(wire
 		(pts
-			(xy 38.1 175.26) (xy 45.72 175.26)
-		)
-		(stroke
-			(width 0)
-			(type default)
-		)
-	)
-	(wire
-		(pts
 			(xy 187.96 86.36) (xy 193.04 86.36)
 		)
@@
 	(wire
 		(pts
-			(xy 38.1 177.8) (xy 45.72 177.8)
-		)
-		(stroke
-			(width 0)
-			(type default)
-		)
-	)
-	(wire
-		(pts
 			(xy 144.78 101.6) (xy 149.86 101.6)
 		)
@@
 	(wire
 		(pts
-			(xy 38.1 170.18) (xy 45.72 170.18)
+			(xy 82.55 185.42) (xy 90.17 185.42)
 		)
 		(stroke
@@
 		(pts
 			(xy 144.78 74.93) (xy 148.59 74.93)
-		)
-		(stroke
-			(width 0)
-			(type default)
-		)
-	)
-	(wire
-		(pts
-			(xy 38.1 182.88) (xy 45.72 182.88)
 		)
 		(stroke
@@
 		)
 	)
-	(label "14V8_DRIVE_OUT"
-		(at 38.1 180.34 180)
-		(effects
-			(font
-				(size 1.27 1.27)
-			)
-			(justify right bottom)
-		)
-	)
 	(label "DRIVE_READ"
 		(at 82.55 180.34 180)
@@
 		)
 	)
-	(label "14V8_COMMS_OUT"
-		(at 38.1 182.88 180)
-		(effects
-			(font
-				(size 1.27 1.27)
-			)
-			(justify right bottom)
-		)
-	)
 	(label "SCL"
 		(at 187.96 69.85 180)
@@
 		)
 	)
-	(label "14V8_DRILL_OUT"
-		(at 38.1 177.8 180)
-		(effects
-			(font
-				(size 1.27 1.27)
-			)
-			(justify right bottom)
-		)
-	)
 	(label "SCL"
-		(at 38.1 170.18 180)
+		(at 82.55 185.42 180)
 		(effects
 			(font
@@
 		)
 	)
-	(label "14V8_ARM_OUT"
-		(at 38.1 175.26 180)
-		(effects
-			(font
-				(size 1.27 1.27)
-			)
-			(justify right bottom)
-		)
-	)
 	(label "SDA"
-		(at 38.1 172.72 180)
+		(at 82.55 187.96 180)
 		(effects
 			(font
@@
 	)
 	(label "14V8_PROTECTED"
-		(at 38.1 185.42 180)
+		(at 83.82 171.45 180)
 		(effects
 			(font
@@
 			)
 			(justify left bottom)
-		)
-	)
-	(hierarchical_label "14V8_DRIVE_OUT"
-		(shape output)
-		(at 45.72 180.34 0)
-		(effects
-			(font
-				(size 1.27 1.27)
-			)
-			(justify left)
 		)
 	)
@@
 		)
 	)
-	(hierarchical_label "14V8_DRILL_OUT"
-		(shape output)
-		(at 45.72 177.8 0)
-		(effects
-			(font
-				(size 1.27 1.27)
-			)
-			(justify left)
-		)
-	)
-	(hierarchical_label "14V8_COMMS_OUT"
-		(shape output)
-		(at 45.72 182.88 0)
-		(effects
-			(font
-				(size 1.27 1.27)
-			)
-			(justify left)
-		)
-	)
 	(hierarchical_label "SCL"
 		(shape output)
-		(at 45.72 170.18 0)
+		(at 90.17 185.42 0)
 		(effects
 			(font
@@
 	(hierarchical_label "SDA"
 		(shape output)
-		(at 45.72 172.72 0)
+		(at 90.17 187.96 0)
 		(effects
 			(font
@@
 	(hierarchical_label "14V8_PROTECTED"
 		(shape input)
-		(at 45.72 185.42 0)
+		(at 90.17 171.45 0)
 		(effects
 			(font
@@
 		(shape output)
 		(at 90.17 177.8 0)
-		(effects
-			(font
-				(size 1.27 1.27)
-			)
-			(justify left)
-		)
-	)
-	(hierarchical_label "14V8_ARM_OUT"
-		(shape output)
-		(at 45.72 175.26 0)
 		(effects
 			(font
@@
 			)
 		)
-		(property "Footprint" "IPRL_footprints:SOP50P490X110-10N"
+		(property "Footprint" "iprl_footprints:SOP50P490X110-10N"
 			(at 140.97 188.9 0)
 			(effects
@@
 			)
 		)
-		(property "Footprint" "IPRL_footprints:SOP50P490X110-10N"
+		(property "Footprint" "iprl_footprints:SOP50P490X110-10N"
 			(at 140.97 162.23 0)
 			(effects

Commit message: corrected power to main
Parts:
- J11, J13, J14: footprint Connector_JST:JST_PH_S4B-PH-K_1x04_P2.00mm_Horizontal -> Connector_JST:JST_GH_SM04B-GHS-TB_1x04-1MP_P1.25mm_Horizontal
Changed lines of the file:
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@@
 			)
 		)
-		(property "Footprint" "Connector_JST:JST_PH_S4B-PH-K_1x04_P2.00mm_Horizontal"
+		(property "Footprint" "Connector_JST:JST_GH_SM04B-GHS-TB_1x04-1MP_P1.25mm_Horizontal"
 			(at 198.12 72.39 0)
 			(effects
@@
 			)
 		)
-		(property "Footprint" "Connector_JST:JST_PH_S4B-PH-K_1x04_P2.00mm_Horizontal"
+		(property "Footprint" "Connector_JST:JST_GH_SM04B-GHS-TB_1x04-1MP_P1.25mm_Horizontal"
 			(at 198.12 83.82 0)
 			(effects
@@
 			)
 		)
-		(property "Footprint" "Connector_JST:JST_PH_S4B-PH-K_1x04_P2.00mm_Horizontal"
+		(property "Footprint" "Connector_JST:JST_GH_SM04B-GHS-TB_1x04-1MP_P1.25mm_Horizontal"
 			(at 198.12 95.25 0)
 			(effects

Commit message: a 5 hour binge of PCB layout on the main
Parts:
- removed J14: Conn_01x04, Connector_JST:JST_GH_SM04B-GHS-TB_1x04-1MP_P1.25mm_Horizontal, symbol Connector_Generic:Conn_01x04
Connections:
- net +3.3V: now also IC2.1 (ADDR); no longer IC3.1 (ADDR)
- net ARM_READ: now also IC3.5 (AIN1); no longer IC3.4 (AIN0)
- net COMMS_READ: now also IC3.4 (AIN0); no longer IC2.6 (AIN2)
- net DRILL_READ: now also IC2.4 (AIN0); no longer IC2.7 (AIN3)
- net DRIVE_READ: now also IC2.5 (AIN1); no longer IC3.5 (AIN1)
- net at R1.2, R3.1: now also IC2.6 (AIN2); no longer IC2.5 (AIN1)
- net at R5.2: now also IC3.1 (ADDR); no longer IC2.1 (ADDR)
Other:
- moved on the sheet: R1, R3, R5
