File: PCBs/Power_V2_main/high_sided_switch.kicad_sch (KiCad schematic)
At the start: 4 parts, among them Q1 BC846, Q2 SiSS27DN

Commit message: follow up changes from meeting
Parts:
- removed Q1: BC846, Package_TO_SOT_SMD:SOT-23, symbol Transistor_BJT:BC846
- removed R19: 1k, Resistor_SMD:R_0805_2012Metric, symbol Device:R
- added Q1: IRLML0030, Package_TO_SOT_SMD:SOT-23, symbol Transistor_FET:IRLML0030
- R24: value 5k -> 5.1k
Connections:
- net CONTROL_IN: now also Q1.1 (G)
- net GATE: now also Q1.3 (D)
- net GND: now also Q1.2 (S)
- net POWER_IN: now also Q2.1 (S), Q2.2 (S), Q2.3 (S); no longer Q2.5 (D)
- net POWER_OUT: now also Q2.5 (D); no longer Q2.1 (S), Q2.2 (S), Q2.3 (S)
