File: PCBs/Power_V2_main/Power_V2_main.kicad_pcb (KiCad board)
At the start: 2 copper layers, 100 x 100 mm, 66 parts, among them IC2 ADS1115BQDGSRQ1, IC3 ADS1115BQDGSRQ1, J10 TYPE-C-31-M-12, J11 Conn_01x04, J12 Conn_01x02, J13 Conn_01x04, J15 Conn_01x04, J18 YK4420203000G, J2 Conn_01x02, J3 Conn_01x02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

Commit message: follow up changes from meeting
Parts:
- removed J15: Conn_01x04, Connector_JST:JST_GH_BM04B-GHS-TBT_1x04-1MP_P1.25mm_Vertical
- removed Q3: BC846, Package_TO_SOT_SMD:SOT-23
- removed R11, R12, R13, R14, R15, R16, R6: 500, Resistor_SMD:R_0805_2012Metric
- removed R17: 1k, Resistor_SMD:R_0805_2012Metric
- added J1: Conn_01x05, Connector_JST:JST_EH_B5B-EH-A_1x05_P2.50mm_Vertical, F.Cu at (239.8, 173.5)
- added Q5: IRLML0030, Package_TO_SOT_SMD:SOT-23, F.Cu at (218.7, 161.8)
- added Q6: IRLML0030, Package_TO_SOT_SMD:SOT-23, F.Cu at (214.7, 161.8)
- added Q7: SiSS27DN, Package_SO:Vishay_PowerPAK_1212-8_Single, F.Cu at (228.9, 175.7)
- D4: value SM15T22A -> SM15T22CA
- H1, H2, H3: footprint MountingHole:MountingHole_2.5mm -> MountingHole:MountingHole_2.7mm_M2.5_DIN965_Pad_TopBottom
- Q1: value BC846 -> IRLML0030
- R18, R24: value 5k -> 5.1k
- R19: value 1k -> 5.1k
- R22, R23: value 5k -> 5k1
- R4: value 500 -> 65; footprint Resistor_SMD:R_0805_2012Metric -> Resistor_THT:R_Axial_DIN0414_L11.9mm_D4.5mm_P15.24mm_Horizontal
- moved R19 14.7 mm to (225.6, 175.7)
- moved U5 13.6 mm to (246.2, 156.2), turned to 0 degrees
- moved G*** 6.38 mm to (251.6, 171.2), turned to 90 degrees
- moved R24 4.53 mm to (231.8, 167.8), turned to -90 degrees
- moved D1 3.92 mm to (246.9, 147.9), turned to -90 degrees
- moved Q4 3.65 mm to (232.5, 171.8), turned to 0 degrees
- moved Q1 3.20 mm to (222.7, 161.8), turned to -90 degrees
- moved R4 3.08 mm to (247.7, 143.8), turned to 0 degrees
- moved D4 1.10 mm to (251.1, 151.5)
- moved R18 0.95 mm to (229.2, 171.8), turned to -90 degrees
- moved Q2 0.49 mm to (235.1, 167.8), turned to 0 degrees
- turned R1 to 90 degrees
- turned R3 to -90 degrees
Connections:
- Q1 pad 1: /LED Indicators/Green switch/BASE -> /Control/IND_GREEN
- Q2 pad 1: /LED Indicators/GREEN_OUT -> /14V8_PROTECTED
- Q2 pad 2: /LED Indicators/GREEN_OUT -> /14V8_PROTECTED
- Q2 pad 3: /LED Indicators/GREEN_OUT -> /14V8_PROTECTED
- Q2 pad 5: /14V8_PROTECTED -> /LED Indicators/GREEN_OUT
- Q4 pad 1: /LED Indicators/YELLOW_OUT -> /14V8_PROTECTED
- Q4 pad 2: /LED Indicators/YELLOW_OUT -> /14V8_PROTECTED
- Q4 pad 3: /LED Indicators/YELLOW_OUT -> /14V8_PROTECTED
- Q4 pad 5: /14V8_PROTECTED -> /LED Indicators/YELLOW_OUT
- R19 pad 1: /Control/IND_GREEN -> /14V8_PROTECTED
- R19 pad 2: /LED Indicators/Green switch/BASE -> /LED Indicators/Siren switch/GATE
- U1 pad 15: /Control/IND_YELLOW -> /Control/IND_SIREN
- U1 pad 18: unconnected-(U1-IO10-Pad18) -> /Control/IND_YELLOW
Routing:
- net /LED Indicators/Siren switch/GATE: track 0.00 -> 18.6 mm, vias 0 -> 2
- net Net-(J12-Pin_2): track 20.5 -> 7.00 mm
- net /LED Indicators/SIREN_OUT: track 0.00 -> 13.4 mm
- net /Protection and power/EMERG_OUT: track 29.5 -> 16.8 mm
- net /LED Indicators/YELLOW_OUT: track 22.1 -> 9.70 mm
- net /LED Indicators/Green switch/GATE: track 20.7 -> 13.7 mm
- net /LED Indicators/GREEN_OUT: track 13.0 -> 6.06 mm
- net /LED Indicators/Yellow switch/GATE: track 19.4 -> 16.1 mm
- net /Control/IND_SIREN: track 0.00 -> 3.05 mm
- net /LED Indicators/Yellow switch/BASE: track 1.89 -> 0.00 mm
- net /LED Indicators/Green switch/BASE: track 1.75 -> 0.00 mm
- net /14V8_PROTECTED: track 8.82 -> 7.13 mm, vias 1 -> 0
- net Net-(IC2-AIN2): track 7.22 -> 5.58 mm
- net GND: track 116.2 -> 115.9 mm, vias 13 -> 15
Other:
- board text added: "GREEN YELLOW SIREN GND RED"
- board text added: "SCL SDA VDD GND"

Commit message: main board ordered
Parts:
- added J14: Conn_01x04, Connector_JST:JST_GH_BM04B-GHS-TBT_1x04-1MP_P1.25mm_Vertical, F.Cu at (235.5, 178.5)
- J1: value Conn_01x05 -> Conn_01x04; footprint Connector_JST:JST_EH_B5B-EH-A_1x05_P2.50mm_Vertical -> Connector_JST:JST_GH_BM04B-GHS-TBT_1x04-1MP_P1.25mm_Vertical
- moved J1 9.25 mm to (241.8, 164.5), turned to -90 degrees
Connections:
- J1 pad 3: /LED Indicators/SIREN_OUT -> /LED Indicators/GREEN_OUT
Routing:
- net /LED Indicators/SIREN_OUT: track 13.4 -> 4.54 mm
- net GND: track 115.9 -> 122.0 mm, vias 15 -> 18
- net /LED Indicators/Yellow switch/GATE: track 16.1 -> 14.7 mm
- net /LED Indicators/GREEN_OUT: track 6.06 -> 5.39 mm
Other:
- board text added: "RED GND GREEN YELLOW"
- board text added: "SIREN GND 14V8 GND"
- board text removed: "GREEN YELLOW SIREN GND RED"
