File: PCBs/Arm Schematic V2/Arm Schematic V2/Arm Schematic V2.kicad_sch (KiCad schematic)
At the start: 94 parts, among them J1 Conn_01x03, J10 Conn_01x04, J11 Conn_01x04, J12 Conn_01x02, J13 Conn_01x04, J14 Conn_01x03, J15 Conn_01x03, J16 Conn_01x02, J17 Conn_01x02, J18 Conn_01x02, J19 Conn_01x02, J2 Conn_01x04, J3 Conn_01x04, J4 Conn_01x04, J5 Conn_01x02, J6 Conn_01x04, J7 Conn_01x04, J8 Conn_01x04, J9 Conn_01x04, Q1 BSS138, Q10 BSS138, Q11 BSS138, Q12 BSS138, Q2 BSS138, Q3 BSS138, Q4 BSS138, Q5 BSS138, Q6 BSS138, Q7 BSS138, Q8 BSS138, Q9 BSS138, U1 AMS1117-3.3, U3 ADS1115IDGS, U8 TCA9548APWR

Commit message: drc clean arm v2
Parts:
- removed J12: Conn_01x02, Connector_JST:JST_GH_BM02B-GHS-TBT_1x02-1MP_P1.25mm_Vertical, symbol Connector_Generic:Conn_01x02
- removed R1: 5.1k, Resistor_SMD:R_0805_2012Metric, symbol Device:R
- removed R2: 10k, Resistor_SMD:R_0805_2012Metric, symbol Device:R
- added J20: Conn_01x04, Connector_JST:JST_GH_BM04B-GHS-TBT_1x04-1MP_P1.25mm_Vertical, symbol Connector_Generic:Conn_01x04
- added R50: 0R, Resistor_SMD:R_0805_2012Metric, symbol Device:R
Connections:
- net PLUG is gone; now on net GND: J1.3 (Pin_3)
- net +3.3V: now also J1.2 (Pin_2), J20.3 (Pin_3), R50.1
- net +5P: no longer J1.1 (Pin_1)
- net ESP_SCL: now also J20.1 (Pin_1)
- net ESP_SDA: now also J20.2 (Pin_2)
- net GND: now also J20.4 (Pin_4); no longer J1.2 (Pin_2)
- net at U2.1 (3.3V): now also R50.2
- net AIN0 renamed PH_reading
- net PH_reading: now also J1.1 (Pin_1)
- no-connect marks 13 -> 12
