File: PCBs/Arm Schematic V2/Arm Schematic V2/Arm Schematic V2.kicad_pcb (KiCad board)
At the start: 2 copper layers, 100 x 80 mm, 93 parts, among them J1 Conn_01x03, J10 Conn_01x04, J11 Conn_01x04, J13 Conn_01x04, J14 Conn_01x03, J15 Conn_01x03, J16 Conn_01x02, J17 Conn_01x02, J18 Conn_01x02, J19 Conn_01x02, J2 Conn_01x04, J3 Conn_01x04, J4 Conn_01x04, J5 Conn_01x02, J6 Conn_01x04, J7 Conn_01x04, J8 Conn_01x04, J9 Conn_01x04, Q1 BSS138, Q10 BSS138, Q11 BSS138, Q12 BSS138, Q2 BSS138, Q3 BSS138, Q4 BSS138, Q5 BSS138, Q6 BSS138, Q7 BSS138, Q8 BSS138, Q9 BSS138, U1 AMS1117-3.3, U3 ADS1115IDGS, U8 TCA9548APWR

Commit message: drc clean arm v2
Parts:
- removed R1: 5.1k, Resistor_SMD:R_0805_2012Metric
- removed R2: 10k, Resistor_SMD:R_0805_2012Metric
- added J20: Conn_01x04, Connector_JST:JST_GH_BM04B-GHS-TBT_1x04-1MP_P1.25mm_Vertical, F.Cu at (58.5, 136.7)
- added R50: 0R, Resistor_SMD:R_0805_2012Metric, F.Cu at (73.8, 112.8)
- moved J1 3.85 mm to (48.4, 136.7)
- moved U2 0.12 mm to (80.0, 112.4)
Connections:
- J1 pad 1: +5P -> /PH_reading
- J1 pad 2: GND -> +3.3V
- J1 pad 3: /PLUG -> GND
- U2 pad 1: unconnected-(U2-3.3V-Pad1) -> Net-(U2-3.3V)
- U3 pad 4: /AIN0 -> /PH_reading
Routing:
- net +5P: track 299.5 -> 251.7 mm
- net +3.3V: track 379.2 -> 407.2 mm
- net GND: track 21.4 -> 47.9 mm
- net /ESP_SCL: track 57.1 -> 75.6 mm, vias 1 -> 3
- net /ESP_SDA: track 66.3 -> 80.8 mm, vias 2 -> 4
- net /PH_reading: track 0.00 -> 11.2 mm
- net /AIN0: track 8.05 -> 0.00 mm
- net /ENA_1: track 63.8 -> 56.3 mm
- net /DIR_1: track 63.2 -> 55.6 mm
- net /PUL_1: track 62.0 -> 55.0 mm
- net /ENA_0: track 61.0 -> 54.1 mm
- net /DIR_0: track 59.3 -> 53.4 mm
- net Net-(U2-3.3V): track 0.00 -> 5.46 mm
- net /PLUG: track 4.74 -> 0.00 mm
- net /IN2: track 23.3 -> 26.1 mm
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Other:
- board text added: "I2C output"
- board text added: "pH Sensor"
- board text removed: "PH Sensor"

Commit message: moved via out the pad, don't worry we like you Samuel
Routing:
- net GND: track 47.9 -> 50.1 mm
Changed lines of the file:
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@@
-	)
-	(segment
-		(start 114.35 65.5)
-		(end 114.35 65.65)
-		(width 0.2)
-		(layer "F.Cu")
-		(net 1)
-	)
-	(segment
-		(start 60.775 102.475)
-		(end 60.75 102.5)
-		(width 0.2)
-		(layer "F.Cu")
-		(net 1)
 	)
 	(segment
@@
 	)
 	(segment
+		(start 60.775 102.475)
+		(end 61.7625 102.475)
+		(width 0.2)
+		(layer "F.Cu")
+		(net 1)
+	)
+	(segment
 		(start 89.917856 133.817856)
 		(end 89.917856 134.7)
@@
 	)
 	(segment
+		(start 60.7125 102.586673)
+		(end 60.7125 102.5375)
+		(width 0.2)
+		(layer "F.Cu")
+		(net 1)
+	)
+	(segment
 		(start 57.6 101.4)
 		(end 57.184491 101.4)
@@
 	)
 	(segment
+		(start 115.6 66.9)
+		(end 114.35 65.65)
+		(width 0.2)
+		(layer "F.Cu")
+		(net 1)
+	)
+	(segment
 		(start 56.0375 100.2875)
 		(end 56.0375 100.525)
@@
 	)
 	(segment
+		(start 115.6 67.4)
+		(end 115.6 66.9)
+		(width 0.2)
+		(layer "F.Cu")
+		(net 1)
+	)
+	(segment
 		(start 35.23125 109.01875)
 		(end 34.95 109.01875)
@@
 	)
 	(segment
-		(start 114.35 65.65)
-		(end 114.25 65.75)
+		(start 60.7125 102.5375)
+		(end 60.775 102.475)
 		(width 0.2)
 		(layer "F.Cu")
@@
 	)
 	(segment
+		(start 114.35 65.65)
+		(end 114.35 65.5)
+		(width 0.2)
+		(layer "F.Cu")
+		(net 1)
+	)
+	(segment
 		(start 54 121.3875)
 		(end 53 120.3875)
@@
 	)
 	(segment
-		(start 61.7625 102.475)
-		(end 60.775 102.475)
-		(width 0.2)
-		(layer "F.Cu")
-		(net 1)
-	)
-	(segment
 		(start 74.9 133.8)
 		(end 74.875 133.825)
@@
 	)
 	(via
-		(at 60.75 102.5)
+		(at 60.7125 102.586673)
 		(size 0.6)
 		(drill 0.3)
@@
 	)
 	(via
-		(at 114.25 65.75)
+		(at 115.6 67.4)
 		(size 0.6)
 		(drill 0.3)
@@
 	)
 	(segment
+		(start 98.4 65.6)
+		(end 98.5 65.5)
+		(width 0.4)
+		(layer "F.Cu")
+		(net 3)
+	)
+	(segment
 		(start 50.544013 70)
 		(end 58.175 70)
@@
 	)
 	(segment
-		(start 98.02727 70)
-		(end 98.02727 65.97273)
-		(width 0.4)
-		(layer "F.Cu")
-		(net 3)
-	)
-	(segment
 		(start 86.071589 70)
 		(end 86.071589 69.828411)
@@
 	)
 	(segment
-		(start 98.02727 65.97273)
-		(end 98.5 65.5)
-		(width 0.4)
-		(layer "F.Cu")
-		(net 3)
-	)
-	(segment
 		(start 62.062499 64.25)
 		(end 62.4625 64.650001)
@@
 	)
 	(segment
+		(start 98.4 69.62727)
+		(end 98.4 65.6)
+		(width 0.4)
+		(layer "F.Cu")
+		(net 3)
+	)
+	(segment
 		(start 74.115908 70)
 		(end 74.115908 65.609092)
@@
 		(width 0.4)
 		(layer "F.Cu")
+		(net 3)
+	)
+	(segment
+		(start 98.02727 70)
+		(end 98.4 69.62727)
+		(width 0.4)
+		(layer "F.Cu")

Commit message: drc clean boards
Parts:
- added G***: LOGO, IPRL Footprints:IPRL_31mm, B.Cu at (111.1, 99.7)
