File: PCBs/encoder/encoder.kicad_pcb (KiCad board)
At the start: 2 copper layers, 23 x 23 mm, 17 parts, among them J1 Conn_01x04, J2 Conn_01x04, J3 Conn_01x04, U1 AS5600-ASOT, U2 STM32G031G6Ux

Commit message: fix encoder board fuck you ben
Connections:
- J1 pad 1: +3V3 -> GND
- J1 pad 2: GND -> +3V3
- J2 pad 1: +3V3 -> GND
- J2 pad 2: GND -> +3V3
