File: PCBs/Drive board V5/iprld.kicad_sch (KiCad schematic)
At the start: 16 parts, among them J1 Conn_01x02, J2 Conn_02x01, J3 Conn_02x02_Top_Bottom, U1 TJA1051T-3, U15 AMS1117-3.3

Commit message: Updated drive board
Parts:
- removed C14, C26: 10u, Capacitor_SMD:C_0805_2012Metric, symbol Device:C
- removed C15: 1u, Capacitor_SMD:C_0805_2012Metric, symbol Device:C
- removed C21: 0.1u, Capacitor_SMD:C_0805_2012Metric, symbol Device:C
- removed U15: AMS1117-3.3, Package_TO_SOT_SMD:SOT-223-3_TabPin2, symbol Regulator_Linear:AMS1117-3.3
- added C3: 0.1u, Capacitor_SMD:C_0805_2012Metric, symbol Device:C
Connections:
- net +5V: now also C3.1
- net GND: now also C3.2
- net CANH renamed CAN_P
- net CANL renamed CAN_N
Other:
- note removed: "5V -> 3.3V conversion"
- moved on the sheet: C1, J1

Commit message: Drive v5 changes
Other:
- moved on the sheet: H1, H2, H3, H4
Changed lines of the file:
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@@
 	(symbol
 		(lib_id "Mechanical:MountingHole")
-		(at 269.24 237.49 0)
+		(at 223.52 40.64 0)
 		(unit 1)
 		(exclude_from_sim yes)
@@
 		(fields_autoplaced yes)
 		(property "Reference" "H3"
-			(at 271.78 236.2199 0)
+			(at 226.06 39.3699 0)
 			(effects
 				(font
@@
 		)
 		(property "Value" "MountingHole"
-			(at 271.78 238.7599 0)
+			(at 226.06 41.9099 0)
 			(effects
 				(font
@@
 		)
 		(property "Footprint" "MountingHole:MountingHole_3.2mm_M3_Pad_TopBottom"
-			(at 269.24 237.49 0)
+			(at 223.52 40.64 0)
 			(effects
 				(font
@@
 		)
 		(property "Datasheet" "~"
-			(at 269.24 237.49 0)
+			(at 223.52 40.64 0)
 			(effects
 				(font
@@
 		)
 		(property "Description" "Mounting Hole without connection"
-			(at 269.24 237.49 0)
+			(at 223.52 40.64 0)
 			(effects
 				(font
@@
 	(symbol
 		(lib_id "Mechanical:MountingHole")
-		(at 269.24 231.14 0)
+		(at 223.52 34.29 0)
 		(unit 1)
 		(exclude_from_sim yes)
@@
 		(fields_autoplaced yes)
 		(property "Reference" "H2"
-			(at 271.78 229.8699 0)
+			(at 226.06 33.0199 0)
 			(effects
 				(font
@@
 		)
 		(property "Value" "MountingHole"
-			(at 271.78 232.4099 0)
+			(at 226.06 35.5599 0)
 			(effects
 				(font
@@
 		)
 		(property "Footprint" "MountingHole:MountingHole_3.2mm_M3_Pad_TopBottom"
-			(at 269.24 231.14 0)
+			(at 223.52 34.29 0)
 			(effects
 				(font
@@
 		)
 		(property "Datasheet" "~"
-			(at 269.24 231.14 0)
+			(at 223.52 34.29 0)
 			(effects
 				(font
@@
 		)
 		(property "Description" "Mounting Hole without connection"
-			(at 269.24 231.14 0)
+			(at 223.52 34.29 0)
 			(effects
 				(font
@@
 	(symbol
 		(lib_id "Mechanical:MountingHole")
-		(at 269.24 243.84 0)
+		(at 223.52 46.99 0)
 		(unit 1)
 		(exclude_from_sim yes)
@@
 		(fields_autoplaced yes)
 		(property "Reference" "H4"
-			(at 271.78 242.5699 0)
+			(at 226.06 45.7199 0)
 			(effects
 				(font
@@
 		)
 		(property "Value" "MountingHole"
-			(at 271.78 245.1099 0)
+			(at 226.06 48.2599 0)
 			(effects
 				(font
@@
 		)
 		(property "Footprint" "MountingHole:MountingHole_3.2mm_M3_Pad_TopBottom"
-			(at 269.24 243.84 0)
+			(at 223.52 46.99 0)
 			(effects
 				(font
@@
 		)
 		(property "Datasheet" "~"
-			(at 269.24 243.84 0)
+			(at 223.52 46.99 0)
 			(effects
 				(font
@@
 		)
 		(property "Description" "Mounting Hole without connection"
-			(at 269.24 243.84 0)
+			(at 223.52 46.99 0)
 			(effects
 				(font
@@
 	(symbol
 		(lib_id "Mechanical:MountingHole")
-		(at 269.24 223.52 0)
+		(at 223.52 26.67 0)
 		(unit 1)
 		(exclude_from_sim yes)
@@
 		(fields_autoplaced yes)
 		(property "Reference" "H1"
-			(at 271.78 222.2499 0)
+			(at 226.06 25.3999 0)
 			(effects
 				(font
@@
 		)
 		(property "Value" "MountingHole"
-			(at 271.78 224.7899 0)
+			(at 226.06 27.9399 0)
 			(effects
 				(font
@@
 		)
 		(property "Footprint" "MountingHole:MountingHole_3.2mm_M3_Pad_TopBottom"
-			(at 269.24 223.52 0)
+			(at 223.52 26.67 0)
 			(effects
 				(font
@@
 		)
 		(property "Datasheet" "~"
-			(at 269.24 223.52 0)
+			(at 223.52 26.67 0)
 			(effects
 				(font
@@
 		)
 		(property "Description" "Mounting Hole without connection"
-			(at 269.24 223.52 0)
-			(effects
-				(font
+			(at 223.52 26.67 0)
+			(effects
+				(font

Commit message: Updates drive board
Other:
- note removed: "-keep traces short for the clock, keep caps close"
- note removed: "NOTES: -check if all I2C connection is correct - pull up resistors etc no pull up R. required on the multiplexer - it has internal pull ups"
Changed lines of the file:
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@@
-		)
-	)
-	(text "NOTES:\n\n-check if all I2C connection is correct - pull up resistors etc\n	no pull up R. required on the multiplexer - it has internal pull ups\n\n"
-		(exclude_from_sim no)
-		(at 305.816 372.11 0)
-		(effects
-			(font
-				(size 1.27 1.27)
-			)
 		)
 	)
@@
 		(effects
 			(font
-				(size 1.27 1.27)
-			)
-		)
-	)
-	(text "\n-keep traces short for the clock, keep caps close\n"
-		(exclude_from_sim no)
-		(at 305.562 379.984 0)
-		(effects
-			(font

Commit message: Fixed drive board
had pwm on input only pins :(
Connections:
- net M1: now also U2.10 (GPIO26); no longer U2.6 (GPIO35)
- net M4: now also U2.9 (GPIO25); no longer U2.5 (GPIO34)
Changed lines of the file:
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@@
+	)
+	(no_connect
+		(at 149.86 36.83)
 	)
 	(no_connect
@@
 	)
 	(no_connect
+		(at 149.86 39.37)
+	)
+	(no_connect
 		(at 185.42 57.15)
 	)
@@
 	)
 	(no_connect
-		(at 149.86 46.99)
-	)
-	(no_connect
 		(at 149.86 54.61)
 	)
@@
 	)
 	(no_connect
-		(at 149.86 49.53)
-	)
-	(no_connect
 		(at 149.86 34.29)
 	)
@@
 	(wire
 		(pts
-			(xy 146.05 36.83) (xy 149.86 36.83)
-		)
-		(stroke
-			(width 0)
-			(type default)
-		)
-	)
-	(wire
-		(pts
 			(xy 143.51 72.39) (xy 149.86 72.39)
 		)
@@
 	(wire
 		(pts
+			(xy 146.05 49.53) (xy 149.86 49.53)
+		)
+		(stroke
+			(width 0)
+			(type default)
+		)
+	)
+	(wire
+		(pts
 			(xy 96.52 92.71) (xy 99.06 92.71)
 		)
@@
 	(wire
 		(pts
+			(xy 146.05 46.99) (xy 149.86 46.99)
+		)
+		(stroke
+			(width 0)
+			(type default)
+		)
+	)
+	(wire
+		(pts
 			(xy 189.23 39.37) (xy 185.42 39.37)
 		)
@@
 		(pts
 			(xy 29.21 96.52) (xy 29.21 99.06)
-		)
-		(stroke
-			(width 0)
-			(type default)
-		)
-	)
-	(wire
-		(pts
-			(xy 146.05 39.37) (xy 149.86 39.37)
 		)
 		(stroke
@@
 		)
 	)
+	(label "M4"
+		(at 146.05 46.99 0)
+		(effects
+			(font
+				(size 1.27 1.27)
+			)
+			(justify left bottom)
+		)
+	)
 	(label "M1"
 		(at 96.52 92.71 0)
@@
 		)
 	)
+	(label "M1"
+		(at 146.05 49.53 0)
+		(effects
+			(font
+				(size 1.27 1.27)
+			)
+			(justify left bottom)
+		)
+	)
 	(label "CAN_TX"
 		(at 33.02 109.22 0)
@@
 		)
 	)
-	(label "M1"
-		(at 146.05 39.37 0)
-		(effects
-			(font
-				(size 1.27 1.27)
-			)
-			(justify left bottom)
-		)
-	)
 	(label "CAN_TX"
 		(at 189.23 39.37 0)
 		(effects
 			(font
-				(size 1.27 1.27)
-			)
-			(justify left bottom)
-		)
-	)
-	(label "M4"
-		(at 146.05 36.83 0)
-		(effects
-			(font

Commit message: Added termination resistor to drive
Can be used in event that drive board is used as one end of can bus
Parts:
- added R1: 120, Resistor_SMD:R_0805_2012Metric, symbol Device:R
Connections:
- net CAN_N: now also R1.2
- net CAN_P: now also R1.1
Changed lines of the file:
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@@
+	(wire
+		(pts
+			(xy 76.2 118.11) (xy 78.74 118.11)
+		)
+		(stroke
+			(width 0)
+			(type default)
+		)
+	)
 	(wire
 		(pts
@@
 	(wire
 		(pts
+			(xy 76.2 110.49) (xy 76.2 111.76)
+		)
+		(stroke
+			(width 0)
+			(type default)
+		)
+	)
+	(wire
+		(pts
 			(xy 146.05 46.99) (xy 149.86 46.99)
 		)
@@
 	(wire
 		(pts
+			(xy 76.2 116.84) (xy 76.2 118.11)
+		)
+		(stroke
+			(width 0)
+			(type default)
+		)
+	)
+	(wire
+		(pts
 			(xy 147.32 26.67) (xy 149.86 26.67)
 		)
@@
 	(wire
 		(pts
+			(xy 76.2 111.76) (xy 66.04 111.76)
+		)
+		(stroke
+			(width 0)
+			(type default)
+		)
+	)
+	(wire
+		(pts
+			(xy 78.74 110.49) (xy 76.2 110.49)
+		)
+		(stroke
+			(width 0)
+			(type default)
+		)
+	)
+	(wire
+		(pts
 			(xy 25.4 116.84) (xy 40.64 116.84)
 		)
@@
 		(pts
 			(xy 49.53 34.29) (xy 53.34 34.29)
+		)
+		(stroke
+			(width 0)
+			(type default)
+		)
+	)
+	(wire
+		(pts
+			(xy 66.04 116.84) (xy 76.2 116.84)
 		)
 		(stroke
@@
 					(unit 1)
 				)
+			)
+		)
+	)
+	(symbol
+		(lib_id "Device:R")
+		(at 78.74 114.3 0)
+		(unit 1)
+		(exclude_from_sim no)
+		(in_bom yes)
+		(on_board yes)
+		(dnp no)
+		(fields_autoplaced yes)
+		(property "Reference" "R1"
+			(at 81.28 113.0299 0)
+			(effects
+				(font
+					(size 1.27 1.27)
+				)
+				(justify left)
+			)
+		)
+		(property "Value" "120"
+			(at 81.28 115.5699 0)
+			(effects
+				(font
+					(size 1.27 1.27)
+				)
+				(justify left)
+			)
+		)
+		(property "Footprint" "Resistor_SMD:R_0805_2012Metric"
+			(at 76.962 114.3 90)
+			(effects
+				(font
+					(size 1.27 1.27)
+				)
+				(hide yes)
+			)
+		)
+		(property "Datasheet" "~"
+			(at 78.74 114.3 0)
+			(effects
+				(font
+					(size 1.27 1.27)
+				)
+				(hide yes)
+			)
+		)
+		(property "Description" "Resistor"
+			(at 78.74 114.3 0)
+			(effects
+				(font
+					(size 1.27 1.27)
+				)
+				(hide yes)
+			)
+		)
+		(pin "2"
+		)
+		(pin "1"
+		)
+		(instances
+			(project ""
+				(path "/f88582ba-beb9-4fb5-aa18-f7c4bf4c6866"
+					(reference "R1")
+					(unit 1)
+				)
