File: PCBs/DRILLTEAM/DRILLTEAMYMchanges.kicad_pcb (KiCad board)
At the start: 2 copper layers, 168 x 111.5 mm, 71 parts, among them J1 Conn_01x04, J10 Conn_01x02, J11 Conn_01x08, J12 Conn_01x04, J13 Conn_01x02, J14 Conn_01x04, J15 Conn_01x04, J2 Conn_01x04, J3 Conn_01x03, J4 Conn_01x02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

Commit message: Add files via upload
Parts:
- removed J13, J4, J7, J8: Conn_01x02, 436500200:MOLEX_436500200
- J1, J12, J14, J2, J6, J9: footprint 43650-0400:MOLEX_43650-0400 -> 430450400:MOLEX_430450400
- J11: footprint 436500800:MOLEX_436500800 -> 430450800:MOLEX_430450800
- J15: value Conn_01x04 -> Conn_01x08; footprint 43650-0400:MOLEX_43650-0400 -> 430450800:MOLEX_430450800
- J3: footprint 436500300:MOLEX_436500300 -> 430450400:MOLEX_430450400
- moved J15 156.0 mm to (147.7, 75.0), turned to 90 degrees
- moved H3 126.7 mm to (44.0, 75.5)
- moved J12 118.3 mm to (48.5, 58.5), turned to -90 degrees
- moved R29 105.5 mm to (60.1, 55.7), turned to 90 degrees
- moved R28 102.9 mm to (60.1, 59.6), turned to 90 degrees
- moved C35 102.9 mm to (56.6, 67.2), turned to 90 degrees
- moved C36 97.0 mm to (66.7, 56.7), turned to 90 degrees
- moved R30 94.5 mm to (61.6, 70.7), turned to -90 degrees
- moved R31 91.2 mm to (62.6, 75.1), turned to -90 degrees
- moved Q3 90.8 mm to (67.7, 63.6), turned to -90 degrees
- moved C1 83.9 mm to (128.1, 126.0), turned to 180 degrees
- moved J5 81.9 mm to (128.1, 132.5), turned to 180 degrees
- moved A1 81.0 mm to (105.6, 120.8), turned to 90 degrees
- moved C37 80.9 mm to (74.5, 57.0), turned to -90 degrees
- moved R26 78.1 mm to (135.5, 81.9), turned to 90 degrees
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Connections:
- J15 pad 1: unconnected-(J15-Pad1) -> GND
- J15 pad 2: unconnected-(J15-Pad2) -> /LS1
- J15 pad 3: unconnected-(J15-Pad3) -> /LS2
- J15 pad 4: unconnected-(J15-Pad4) -> GND
- U1 pad 10: /LS4 -> /LS3
- U1 pad 11: /LC1DT -> /M2IB
- U1 pad 12: /LC1CLK -> /M2IA
- U1 pad 13: unconnected-(U1-GPIO12-Pad13) -> /M1IA
- U1 pad 15: /LC2DT -> /M1IB
- U1 pad 16: /LC2CLK -> unconnected-(U1-GPIO9-Pad16)
- U1 pad 17: /LC3DT -> unconnected-(U1-GPIO10-Pad17)
- U1 pad 18: /LC3CLK -> unconnected-(U1-GPIO11-Pad18)
- U1 pad 20: /ENC2B -> unconnected-(U1-GPIO6-Pad20)
- U1 pad 21: /ENC2A -> unconnected-(U1-GPIO7-Pad21)
- U1 pad 26: /ENC1B -> /LC3DT
- U1 pad 27: /ENC1A -> /LC3CLK
- U1 pad 28: /Servo1 -> /LC2DT
- U1 pad 29: /M2IB -> /LC2CLK
- U1 pad 3: unconnected-(U1-GPIOP36-Pad3) -> /ENC2B
- U1 pad 30: /M2IA -> /LC1CLK
- U1 pad 31: /M2P -> /LC1DT
- U1 pad 33: /M1IB -> /Servo1
- U1 pad 34: /M1IA -> unconnected-(U1-GPIO3-Pad34)
- U1 pad 35: /M1P -> unconnected-(U1-GPIO1-Pad35)
- U1 pad 4: unconnected-(U1-GPIO39-Pad4) -> /ENC2A
- U1 pad 5: unconnected-(U1-GPIO34-Pad5) -> /ENC1B
- U1 pad 6: unconnected-(U1-GPIO35-Pad6) -> /ENC1A
- U1 pad 7: /LS1 -> /LS2
- U1 pad 8: /LS2 -> /LS4
- U1 pad 9: /LS3 -> /LS1
Routing:
- net GND: track 23.6 -> 455.2 mm, vias 22 -> 16
- net +3.3V: track 407.3 -> 289.3 mm, vias 8 -> 15
- net /M1P: track 60.5 -> 0.00 mm
- net /M2P: track 60.1 -> 0.00 mm
- net /LS4: track 65.8 -> 33.2 mm
- net /LC2CLK: track 52.1 -> 27.0 mm
- net /M2IA: track 60.2 -> 35.6 mm
- net /LC2DT: track 52.6 -> 29.0 mm
- net /LC1CLK: track 31.9 -> 53.4 mm
- net /M2IB: track 60.4 -> 39.7 mm
- net /M1IA: track 60.7 -> 41.9 mm
- net Net-(A1-B2): track 28.7 -> 10.2 mm
- net /LS3: track 52.3 -> 33.8 mm
- net /ENC1A: track 53.6 -> 37.6 mm
- net /LC1DT: track 32.5 -> 47.6 mm
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- removed copper zone on F.Cu, net GND
Other:
- board size 168 x 111.5 mm -> 120 x 93 mm
