File: PCBs/DRILLTEAM/DRILLTEAMYMchanges.kicad_sch (KiCad schematic)
At the start: 71 parts, among them J1 Conn_01x04, J10 Conn_01x02, J11 Conn_01x08, J12 Conn_01x04, J13 Conn_01x02, J14 Conn_01x04, J15 Conn_01x04, J2 Conn_01x04, J3 Conn_01x03, J4 Conn_01x02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

Commit message: Add files via upload
Parts:
- removed J13, J4, J7, J8: Conn_01x02, 436500200:MOLEX_436500200, symbol 436500200:436500200
- removed J15: Conn_01x04, 43650-0400:MOLEX_43650-0400, symbol 43650-0400:43650-0400
- added J15: Conn_01x08, 430450800:MOLEX_430450800, symbol 430450800:430450800
- J1, J12: footprint 43650-0400:MOLEX_43650-0400 -> 430450400:MOLEX_430450400
- J11: footprint 436500800:MOLEX_436500800 -> 430450800:MOLEX_430450800; symbol 436500800:436500800 -> 430450800:430450800; Check_prices https://www.snapeda.com/parts/436500800/Molex/view-part/?re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 -> https://www.snapeda.com/parts/43045-0800/Molex/view-part/?r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; Description_1 Connector Header Through Hole, Right Angle 8 position 0.118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 -> Header 2 Row Right-Angle Snap-In Lock 8 Pin Tin Plate SMT/G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; MAXIMUM_PACKAGE_HEIGHT 5.57 mm -> 8.77mm; MP 436500800 -> 43045-0800; PARTREV D7 -> G; Purchase-URL (none) -> https://www.snapeda.com/api/url_track_click_mouser/?unipart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; SnapEDA_Link https://www.snapeda.com/parts/436500800/Molex/view-part/?re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 -> https://www.snapeda.com/parts/43045-0800/Molex/view-part/?r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
- J14, J2, J6, J9: footprint 43650-0400:MOLEX_43650-0400 -> 430450400:MOLEX_430450400; symbol 43650-0400:43650-0400 -> 430450400:430450400; Check_prices https://www.snapeda.com/parts/436500400/Molex/view-part/?re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 -> https://www.snapeda.com/parts/430450400/Molex/view-part/?re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; Description_1 Conn Wire to Board HDR 4 POS 3mm Solder RA Thru-Hole 4 Term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 -> Conn Wire to Board HDR 4 POS 3mm Solder RA Side Entry Thru-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; MAXIMUM_PACKAGE_HEIGHT 5.57 mm -> 8.77mm; MP 436500400 -> 430450400; PARTREV D7 -> G; Purchase-URL (none) -> https://www.snapeda.com/api/url_track_click_mouser/?unipart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; SnapEDA_Link https://www.snapeda.com/parts/436500400/Molex/view-part/?re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 -> https://www.snapeda.com/parts/430450400/Molex/view-part/?re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
- J3: footprint 436500300:MOLEX_436500300 -> 430450400:MOLEX_430450400; symbol 436500300:436500300 -> 430450400:430450400; Check_prices https://www.snapeda.com/parts/436500300/Molex/view-part/?re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 -> https://www.snapeda.com/parts/430450400/Molex/view-part/?re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; Description_1 Conn Wire to Board HDR 3Power POS 3mm Solder RA Side Entry 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 -> Conn Wire to Board HDR 4 POS 3mm Solder RA Side Entry Thru-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; MAXIMUM_PACKAGE_HEIGHT 5.57 mm -> 8.77mm; MP 436500300 -> 430450400; PARTREV D7 -> G; Purchase-URL (none) -> https://www.snapeda.com/api/url_track_click_mouser/?unipart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; SnapEDA_Link https://www.snapeda.com/parts/436500300/Molex/view-part/?re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 -> https://www.snapeda.com/parts/430450400/Molex/view-part/?re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
Connections:
- net ENC1A: now also U1.6 (GPIO35); no longer U1.27 (GPIO16)
- net ENC1B: now also U1.5 (GPIO34); no longer U1.26 (GPIO4)
- net ENC2A: now also U1.4 (GPIO39); no longer U1.21 (GPIO7)
- net ENC2B: now also U1.3 (GPIOP36); no longer U1.20 (GPIO6)
- net GND: now also J15.1, J15.4, J15.6, J15.8
- net LC1CLK: now also U1.30 (GPIO18); no longer U1.12 (GPIO14)
- net LC1DT: now also U1.31 (GPIO19); no longer U1.11 (GPIO27)
- net LC2CLK: now also U1.29 (GPIO5); no longer U1.16 (GPIO9)
- net LC2DT: now also U1.28 (GPIO17); no longer U1.15 (GPIO13)
- net LC3CLK: now also U1.27 (GPIO16); no longer U1.18 (GPIO11)
- net LC3DT: now also U1.26 (GPIO4); no longer U1.17 (GPIO10)
- net LS1: now also U1.9 (GPIO25), J15.2; no longer U1.7 (GPIO32)
- net LS2: now also U1.7 (GPIO32), J15.3; no longer U1.8 (GPIO33)
- net LS3: now also U1.10 (GPIO26), J15.5; no longer U1.9 (GPIO25)
- net LS4: now also U1.8 (GPIO33), J15.7; no longer U1.10 (GPIO26)
- net M1IA: now also U1.13 (GPIO12); no longer U1.34 (GPIO3)
- net M1IB: now also U1.15 (GPIO13); no longer U1.33 (GPIO21)
- net M1P: no longer U1.35 (GPIO1)
- net M2IA: now also U1.12 (GPIO14); no longer U1.30 (GPIO18)
- net M2IB: now also U1.11 (GPIO27); no longer U1.29 (GPIO5)
- net M2P: no longer U1.31 (GPIO19)
- net Servo1: now also U1.33 (GPIO21); no longer U1.28 (GPIO17)
- no-connect marks 0 -> 14
Other:
- moved on the sheet: H3, R26, R27, R5, R6
