File: PCBs/Arm_Board_v3/Arm_Board_v3.kicad_pcb (KiCad board)
At the start: 2 copper layers, 80 x 80 mm, 28 parts, among them IC1 MC74ACT125DG, IC2 MC74ACT125DG, IC3 MC74ACT125DG, J1 Conn_01x02, J12 Conn_01x03, J14 Conn_01x03, J15 Conn_01x03, J20 Conn_01x04, J4 Conn_01x03, J5 Conn_01x04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

Commit message: Fixed servo pin and added labels
Connections:
- U2 pad 29: /Servo_2 -> unconnected-(U2-GPIO5-Pad29)
- U2 pad 37: unconnected-(U2-GPIO23-Pad37) -> /Servo_2
Routing:
- net /Servo_2: track 10.8 -> 32.5 mm
Other:
- board text added: "ADC"
- board text added: "I2C"
- board text added: "Servos"
- board text added: "Steppers"
Changed lines of the file:
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@@
 	(net 51 "unconnected-(U2-GPIO2-Pad24)")
 	(net 52 "unconnected-(U2-GPIO13-Pad15)")
-	(net 53 "unconnected-(U2-GPIO23-Pad37)")
+	(net 53 "unconnected-(U2-GPIO5-Pad29)")
 	(footprint "Resistor_SMD:R_0805_2012Metric"
 		(layer "F.Cu")
@@
 			(at 0 -4.15 0)
 			(layer "F.SilkS")
+			(hide yes)
 			(effects
 				(font
@@
 			(layers "*.Cu" "*.Mask")
 			(remove_unused_layers no)
-			(net 23 "/Servo_2")
+			(net 53 "unconnected-(U2-GPIO5-Pad29)")
 			(pinfunction "GPIO5")
 			(pintype "bidirectional")
@@
 			(layers "*.Cu" "*.Mask")
 			(remove_unused_layers no)
-			(net 53 "unconnected-(U2-GPIO23-Pad37)")
+			(net 23 "/Servo_2")
 			(pinfunction "GPIO23")
 			(pintype "bidirectional")
@@
 			(at 0 -4.15 0)
 			(layer "F.SilkS")
+			(hide yes)
 			(effects
 				(font
@@
 		(layer "Edge.Cuts")
 	)
+	(gr_text "Steppers"
+		(at 87.6 86.342858 270)
+		(layer "F.SilkS")
+		(effects
+			(font
+				(size 1.5 1.5)
+				(thickness 0.3)
+				(bold yes)
+			)
+			(justify left bottom)
+		)
+	)
+	(gr_text "Servos"
+		(at 125.7 95.478571 90)
+		(layer "F.SilkS")
+		(effects
+			(font
+				(size 1.5 1.5)
+				(thickness 0.3)
+				(bold yes)
+			)
+			(justify left bottom)
+		)
+	)
 	(gr_text "Arm Board\nby Samuel A-O"
 		(at 120.5 118 0)
@@
 		)
 	)
+	(gr_text "ADC"
+		(at 112.057143 66.1 0)
+		(layer "F.SilkS")
+		(effects
+			(font
+				(size 1.5 1.5)
+				(thickness 0.3)
+				(bold yes)
+			)
+			(justify left bottom)
+		)
+	)
+	(gr_text "I2C"
+		(at 90.9 66.1 0)
+		(layer "F.SilkS")
+		(effects
+			(font
+				(size 1.5 1.5)
+				(thickness 0.3)
+				(bold yes)
+			)
+			(justify left bottom)
+		)
+	)
 	(segment
 		(start 77.13 102.275)
@@
 	)
 	(segment
+		(start 116.237011 102.191)
+		(end 114.799 100.752989)
+		(width 0.2)
+		(layer "F.Cu")
+		(net 23)
+	)
+	(segment
+		(start 127.68 103.5)
+		(end 126.371 102.191)
+		(width 0.2)
+		(layer "F.Cu")
+		(net 23)
+	)
+	(segment
 		(start 127.5 103.68)
 		(end 127.68 103.5)
@@
 	)
 	(segment
-		(start 116.922349 103.68)
-		(end 127.5 103.68)
+		(start 114.799 85.483349)
+		(end 116.922349 83.36)
+		(width 0.2)
+		(layer "F.Cu")
+		(net 23)
+	)
+	(segment
+		(start 126.371 102.191)
+		(end 116.237011 102.191)
+		(width 0.2)
+		(layer "F.Cu")
+		(net 23)
+	)
+	(segment
+		(start 114.799 100.752989)
+		(end 114.799 85.483349)
 		(width 0.2)
 		(layer "F.Cu")
@@
 		(min_thickness 0.2)
 		(filled_areas_thickness no)
-		(fill yes
+		(fill
 			(thermal_gap 0.2)
 			(thermal_bridge_width 0.2)
