File: PCBs/Arm_Board_v3/Arm_Board_v3.kicad_sch (KiCad schematic)
At the start: 29 parts, among them IC1 MC74ACT125DG, IC2 MC74ACT125DG, IC3 MC74ACT125DG, IC4 MC74ACT125DG, J1 Conn_01x02, J12 Conn_01x03, J14 Conn_01x03, J15 Conn_01x03, J20 Conn_01x04, J4 Conn_01x03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

Commit message: Finished arm pcb
Parts:
- removed IC4: MC74ACT125DG, SOIC127P600X175-14N, symbol 74ACT:MC74ACT125DG
- removed J7: Conn_01x04, symbol Connector_Generic:Conn_01x04
- J1: footprint (none) -> Connector_AMASS:AMASS_XT30PW-M_1x02_P2.50mm_Horizontal
- J12, J14, J15, J4: footprint Connector_JST:JST_GH_BM03B-GHS-TBT_1x03-1MP_P1.25mm_Vertical -> Connector_Molex:Molex_Micro-Fit_3.0_43045-0400_2x02_P3.00mm_Horizontal
- J20, J9: footprint Connector_JST:JST_GH_BM04B-GHS-TBT_1x04-1MP_P1.25mm_Vertical -> Connector_Molex:Molex_Micro-Fit_3.0_43045-0400_2x02_P3.00mm_Horizontal
- J5, J6, J8: footprint (none) -> Connector_Molex:Molex_Micro-Fit_3.0_43045-0400_2x02_P3.00mm_Horizontal
Connections:
- net DIR_3 is gone; now on net Servo_1: U2.30 (GPIO18)
- net ENA_3 is gone; now on net Servo_0: U2.31 (GPIO19)
- net PUL_3 is gone; now on net Servo_2: U2.29 (GPIO5)
- net +3.3V: now also J12.3 (Pin_3); no longer J12.2 (Pin_2)
- net DIR_0: now also U2.12 (GPIO14); no longer U2.11 (GPIO27)
- net DIR_1: now also U2.9 (GPIO25); no longer U2.8 (GPIO33)
- net DIR_2: now also U2.26 (GPIO4); no longer U2.27 (GPIO16)
- net ENA_0: now also U2.11 (GPIO27); no longer U2.10 (GPIO26)
- net ENA_1: now also U2.8 (GPIO33); no longer U2.7 (GPIO32)
- net ENA_2: now also U2.27 (GPIO16); no longer U2.28 (GPIO17)
- net GND: now also J12.2 (Pin_2); no longer J12.3 (Pin_3)
- net PUL_0: now also U2.10 (GPIO26); no longer U2.12 (GPIO14)
- net PUL_1: now also U2.7 (GPIO32); no longer U2.9 (GPIO25)
- net PUL_2: now also U2.28 (GPIO17); no longer U2.26 (GPIO4)
- net Servo_0: no longer U2.37 (GPIO23)
- net Servo_1: no longer U2.15 (GPIO13)
- net Servo_2: no longer U2.24 (GPIO2)
Other:
- moved on the sheet: H1, H2, H3, H4, J20, J9

Commit message: Fixed servo pin and added labels
Connections:
- net Servo_2: now also U2.37 (GPIO23); no longer U2.29 (GPIO5)
Changed lines of the file:
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@@
-		)
-	)
-	(label "Servo_2"
-		(at 254 146.05 0)
-		(effects
-			(font
-				(size 1.27 1.27)
-			)
-			(justify left bottom)
 		)
 	)
@@
 		)
 	)
+	(label "Servo_2"
+		(at 254 125.73 0)
+		(effects
+			(font
+				(size 1.27 1.27)
+			)
+			(justify left bottom)
+		)
+	)
